File: board/rev_a.brd (EAGLE design)
At the start: 56 x 25 mm, 47 parts, among them IC3 MCP2551, Q1 Logic level FET, X1 B4B-ZR

Commit message: [board] Working on analog
Parts:
- added R17, R20: 66K 1%, resistor:R0603
- added R18, R19: 22K 1%, resistor:R0603
- added R21: 100R, resistor:R0603
- R14: value 61.9R 1% -> 62R 1%
- R16: value 150K 1% -> 100K 1%
Connections:
- net CAN_RS renamed CAN_SLEEP
- removed net VS/IP_REF: J2.2, OPA1.6, OPA1.7, R13.2
- removed net VS/OPA4_IN+: MCU.22
- new net N$15: OPA1.1, OPA1.2, R21.2
- new net OPA4_IN+: MCU.22, R19.2, R20.1
- new net VGND: J2.2, OPA1.6, OPA1.7, R13.2, R18.1
- net GND: now also R20.2
- net IP: no longer OPA1.1, OPA1.2
- net OPA4_IN-: now also R17.1, R18.2
- net OPA4_OUT: now also R17.2
- net RCAL: now also R21.1
- net VDDA: now also R16.2
- net VS: now also R16.1, R19.1
Changed lines of the file:
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@@
 <layer number="23" name="tOrigins" color="15" fill="1" visible="yes" active="yes"/>
 <layer number="24" name="bOrigins" color="15" fill="1" visible="yes" active="yes"/>
-<layer number="25" name="tNames" color="7" fill="1" visible="yes" active="yes"/>
-<layer number="26" name="bNames" color="7" fill="1" visible="yes" active="yes"/>
+<layer number="25" name="tNames" color="7" fill="1" visible="no" active="yes"/>
+<layer number="26" name="bNames" color="7" fill="1" visible="no" active="yes"/>
 <layer number="27" name="tValues" color="7" fill="1" visible="no" active="yes"/>
 <layer number="28" name="bValues" color="7" fill="1" visible="no" active="yes"/>
@@
 <element name="R10" library="resistor" package="R0603" value="22K 1%" x="-5.5" y="-57"/>
 <element name="R13" library="resistor" package="R0603" value="100K 1%" x="-5.5" y="-62"/>
-<element name="R14" library="resistor" package="R0603" value="61.9R 1%" x="-5.5" y="-67"/>
+<element name="R14" library="resistor" package="R0603" value="62R 1%" x="-5.5" y="-67"/>
 <element name="R15" library="resistor" package="R0603" value="10K 1%" x="-5.5" y="-72"/>
 <element name="C7" library="resistor" package="C0603" value="100nF" x="-5.5" y="-77"/>
-<element name="R16" library="resistor" package="R0603" value="150K 1%" x="-5.5" y="-82"/>
+<element name="R16" library="resistor" package="R0603" value="100K 1%" x="-5.5" y="-82"/>
 <element name="D1" library="zetex" package="SOT323" value="" x="6.5" y="22.75" rot="R180">
 <attribute name="OC_FARNELL" value="unknown" x="6.5" y="22.75" size="1.778" layer="27" font="vector" ratio="15" rot="R180" display="off"/>
@@
 <attribute name="MPN" value="" x="13.5" y="2" size="1.778" layer="27" font="vector" ratio="15" rot="R90" display="off"/>
 </element>
+<element name="R17" library="resistor" package="R0603" value="66K 1%" x="-5.5" y="-87"/>
+<element name="R18" library="resistor" package="R0603" value="22K 1%" x="-5.5" y="-92"/>
+<element name="R19" library="resistor" package="R0603" value="22K 1%" x="-5.5" y="-97"/>
+<element name="R20" library="resistor" package="R0603" value="66K 1%" x="-5.5" y="-102"/>
+<element name="R21" library="resistor" package="R0603" value="100R" x="-5.5" y="-107"/>
 </elements>
 <signals>
@@
 <contactref element="D1" pad="3"/>
 <contactref element="D5" pad="3"/>
+<contactref element="R20" pad="2"/>
+<wire x1="-4.65" y1="-52" x2="-4.65" y2="-102" width="0" layer="19" extent="1-1"/>
 <wire x1="-4.65" y1="-42" x2="-4.65" y2="-52" width="0" layer="19" extent="1-1"/>
 <wire x1="2.35" y1="-22" x2="-4.65" y2="-42" width="0" layer="19" extent="1-1"/>
@@
 <contactref element="J2" pad="6"/>
 <contactref element="C7" pad="2"/>
+<contactref element="R16" pad="1"/>
+<contactref element="R19" pad="1"/>
+<wire x1="-6.35" y1="-82" x2="-6.35" y2="-97" width="0" layer="19" extent="1-1"/>
+<wire x1="-4.65" y1="-77" x2="-6.35" y2="-82" width="0" layer="19" extent="1-1"/>
 <wire x1="46" y1="18.7" x2="-4.65" y2="-77" width="0" layer="19" extent="1-1"/>
 </signal>
@@
 <contactref element="J2" pad="4"/>
 </signal>
-<signal name="VS/IP_REF">
+<signal name="VGND">
 <contactref element="J2" pad="2"/>
 <contactref element="OPA1" pad="6"/>
 <contactref element="OPA1" pad="7"/>
 <contactref element="R13" pad="2"/>
+<contactref element="R18" pad="1"/>
+<wire x1="-4.65" y1="-62" x2="-6.35" y2="-92" width="0" layer="19" extent="1-1"/>
 <wire x1="21.175" y1="11.425" x2="-4.65" y2="-62" width="0" layer="19" extent="1-1"/>
 <wire x1="21.825" y1="11.425" x2="21.175" y2="11.425" width="0" layer="19" extent="1-1"/>
@@
 <contactref element="R7" pad="1"/>
 <contactref element="R14" pad="1"/>
-<contactref element="OPA1" pad="2"/>
-<contactref element="OPA1" pad="1"/>
-<wire x1="20.525" y1="5.575" x2="-6.35" y2="-67" width="0" layer="19" extent="1-1"/>
-<wire x1="21.175" y1="5.575" x2="20.525" y2="5.575" width="0" layer="19" extent="1-1"/>
-<wire x1="29.15" y1="2" x2="21.175" y2="5.575" width="0" layer="19" extent="1-1"/>
+<wire x1="29.15" y1="2" x2="-6.35" y2="-67" width="0" layer="19" extent="1-1"/>
 <wire x1="46" y1="6" x2="29.15" y2="2" width="0" layer="19" extent="1-1"/>
 </signal>
@@
 <wire x1="10.15" y1="10" x2="10.075" y2="12.675" width="0" layer="19" extent="1-1"/>
 </signal>
-<signal name="CAN_RS">
+<signal name="CAN_SLEEP">
 <contactref element="MCU" pad="3"/>
 <contactref element="R3" pad="2"/>
@@
 <signal name="OPA4_IN-">
 <contactref element="MCU" pad="21"/>
-</signal>
-<signal name="VS/OPA4_IN+">
-<contactref element="MCU" pad="22"/>
+<contactref element="R17" pad="1"/>
+<contactref element="R18" pad="2"/>
+<wire x1="-6.35" y1="-87" x2="-4.65" y2="-92" width="0" layer="19" extent="1-1"/>
+<wire x1="28.5" y1="7.75" x2="-6.35" y2="-87" width="0" layer="19" extent="1-1"/>
 </signal>
 <signal name="OPA4_OUT">
 <contactref element="MCU" pad="25"/>
+<contactref element="R17" pad="2"/>
+<wire x1="30" y1="4.75" x2="-4.65" y2="-87" width="0" layer="19" extent="1-1"/>
 </signal>
 <signal name="NRST">
@@
 <contactref element="OPA1" pad="8"/>
 <contactref element="D5" pad="2"/>
-<wire x1="23.5" y1="14.65" x2="31.5" y2="13.25" width="0" layer="19" extent="1-1"/>
-<wire x1="21.95" y1="14.1999" x2="23.5" y2="14.65" width="0" layer="19" extent="1-1"/>
-<wire x1="20.525" y1="11.425" x2="21.95" y2="14.1999" width="0" layer="19" extent="1-1"/>
-<wire x1="14.4" y1="1.35" x2="20.525" y2="11.425" width="0" layer="19" extent="1-1"/>
+<contactref element="R16" pad="2"/>
+<wire x1="14.4" y1="1.35" x2="-4.65" y2="-82" width="0" layer="19" extent="1-1"/>
+<wire x1="20.525" y1="11.425" x2="14.4" y2="1.35" width="0" layer="19" extent="1-1"/>
+<wire x1="21.95" y1="14.1999" x2="20.525" y2="11.425" width="0" layer="19" extent="1-1"/>
+<wire x1="23.5" y1="14.65" x2="21.95" y2="14.1999" width="0" layer="19" extent="1-1"/>
+<wire x1="31.5" y1="13.25" x2="23.5" y2="14.65" width="0" layer="19" extent="1-1"/>
 </signal>
 <signal name="SWCLK">
@@
 <contactref element="J2" pad="5"/>
 <contactref element="R14" pad="2"/>
+<contactref element="R21" pad="1"/>
+<wire x1="-4.65" y1="-67" x2="-6.35" y2="-107" width="0" layer="19" extent="1-1"/>
 <wire x1="-6.35" y1="-57" x2="-4.65" y2="-67" width="0" layer="19" extent="1-1"/>
 <wire x1="46" y1="16.16" x2="-6.35" y2="-57" width="0" layer="19" extent="1-1"/>
@@
 <wire x1="-6.35" y1="-72" x2="-6.35" y2="-77" width="0" layer="19" extent="1-1"/>
 </signal>
+<signal name="OPA4_IN+">
+<contactref element="MCU" pad="22"/>
+<contactref element="R19" pad="2"/>
+<contactref element="R20" pad="1"/>
+<wire x1="-4.65" y1="-97" x2="-6.35" y2="-102" width="0" layer="19" extent="1-1"/>
+<wire x1="28.5" y1="7.25" x2="-4.65" y2="-97" width="0" layer="19" extent="1-1"/>
+</signal>
+<signal name="N$15">
+<contactref element="OPA1" pad="2"/>
+<contactref element="OPA1" pad="1"/>
+<contactref element="R21" pad="2"/>
+<wire x1="20.525" y1="5.575" x2="-4.65" y2="-107" width="0" layer="19" extent="1-1"/>
+<wire x1="21.175" y1="5.575" x2="20.525" y2="5.575" width="0" layer="19" extent="1-1"/>
+</signal>
 </signals>

Commit message: Routed PCB
Parts:
- removed D3, D4: (no value), zetex:SOT323
- removed J1, J2: (no value), SparkFun-Connectors:1X06_LONGPADS
- removed J3: (no value), SparkFun-Connectors:1X04_LOCK
- removed RN1, RN4: 1K, resistor-dil:0603-ARC
- removed S1: (no value), SparkFun-Switches:TACTILE_SWITCH_SMD_5.2MM
- added LED1: LED-APA102, Ai_LED:LED-APA102
- added PAD1, PAD2, PAD3, PAD4, PAD5, PAD6: WIREPADSMD5-2,5, wirepad:5-2,5
- added R22: 68K 0.1%, resistor:R0603
- added R23: 22K 0.1%, resistor:R0603
- added X2, X3: (no value), con-molex-micro-fit-3_0:43045-0400
- added X5: (no value), con-molex-micro-fit-3_0:43045-0200
- C3: device rcl:E2,5-6 -> rcl:E2,5-5
- IC3: value MCP2551 -> MAX3051
- OPA1: value MCP6002 -> MCP6V64; device linear:TSSOP8 -> linear:TSSOP14
- Q1: value Logic level FET -> VND7NV04
- R10, R18, R19, R7: value 22K 1% -> 22K 0.1%
- R13, R16, R6: value 100K 1% -> 100K 0.1%
- R14: value 62R 1% -> 61.9R 0.1%
- R17, R20: value 66K 1% -> 68K 0.1%
- moved R20 124.3 mm to (36.5, 15.0), turned to 270 degrees
- moved R21 122.3 mm to (48.0, 3.00), turned to 180 degrees
- moved R19 120.3 mm to (38.5, 15.0), turned to 90 degrees
- moved R18 114.7 mm to (48.0, 9.50), turned to 90 degrees
- moved R17 113.4 mm to (48.0, 13.0), turned to 90 degrees
- moved R16 102.9 mm to (38.5, 11.0), turned to 270 degrees
- moved R14 102.2 mm to (55.5, 15.0), turned to 90 degrees
- moved C7 97.5 mm to (36.5, 11.0), turned to 90 degrees
- moved R10 96.8 mm to (54.5, 19.0), turned to 180 degrees
- moved R13 95.8 mm to (51.5, 15.0), turned to 270 degrees
- moved R15 89.5 mm to (36.5, 7.00), turned to 270 degrees
- moved C9 70.0 mm to (16.5, 14.5), turned to 270 degrees
- moved R12 66.2 mm to (19.0, 14.5), turned to 90 degrees
- moved C8 51.6 mm to (12.0, 6.50), turned to 270 degrees
- moved R11 47.9 mm to (14.5, 6.50), turned to 90 degrees
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Connections:
- removed net AN2: MCU.11
- removed net AN3: MCU.12
- removed net BUTTON1: MCU.2, S1.1, S1.2
- removed net HEATER_POS: J2.4
- removed net N$1: Q1.1, RN3.2, RN3.8
- removed net N$3: RN1.2, RN1.8
- removed net N$9: RN1.4, RN1.6
- removed net OPA3_OUT: MCU.19, R6.2
- removed net OPA4_OUT: MCU.25, R17.2
- removed net SCL: J3.3, MCU.42, RN1.3
- removed net SDA: J3.4, MCU.43, RN1.1
- new net HEATER_DIAG: MCU.11, Q1.1, RN3.2, RN3.8
- new net N$10: OPA1.5, R22.2, R23.2
- new net NERST_R: MCU.25, OPA1.14, R17.2
- new net PUMP_I: MCU.19, OPA1.8, R6.2
- new net SPI1_CS: MCU.38
- new net SPI1_MISO: MCU.40
- new net SPI1_MOSI: LED1.1, MCU.41
- new net SPI1_SCK: LED1.2, MCU.39
- net 12V: now also PAD3.1, X2.P$2, X3.P$2; no longer J1.6
- net 5V: now also LED1.4; no longer D3.2, D4.2, IC3.3, J3.2
- net AN1: no longer MCU.10
- net DAC2: now also R15.2; no longer OPA1.5
- net GND: now also LED1.3, OPA1.11, R23.1, X2.P$1, X3.P$1; no longer D3.3, D4.3, J1.1, J3.1, OPA1.4, S1.3, S1.4
- net HEATER_NEG: now also PAD4.1; no longer J2.3
- net IP: now also PAD6.1; no longer J2.1
- net OPA3_IN+: now also OPA1.10; no longer MCU.18
- net OPA3_IN-: now also OPA1.9; no longer MCU.20
- net OPA4_IN+: no longer MCU.22
- net OPA4_IN-: no longer MCU.21
- net OUT1: now also X5.P$2; no longer J1.5
- net OUT2: now also X5.P$1; no longer J1.4
- net OUT3: now also X2.P$4, X3.P$4; no longer J1.3, RN4.1, RN4.2
- net OUT3_PROT: no longer D3.1, RN4.7, RN4.8
- net OUT4: now also X2.P$3, X3.P$3; no longer J1.2, RN4.3, RN4.4
- net OUT4_PROT: no longer D4.1, RN4.5, RN4.6
- net RCAL: now also PAD2.1; no longer J2.5
- net TIM1_CH1: no longer R15.2
- net VBAT: now also MCU.10
- net VCC: now also IC3.3; no longer RN1.5, RN1.7
- net VDDA: now also OPA1.4; no longer OPA1.8
- net VGND: now also MCU.12, PAD5.1; no longer J2.2
- net VS: now also PAD1.1; no longer J2.6
Routing:
- net 12V: track 0.00 -> 188.6 mm
- net 5V: track 0.00 -> 80.9 mm, vias 0 -> 2
- net VGND: track 0.00 -> 54.3 mm, vias 0 -> 3
- net VDDA: track 0.00 -> 47.9 mm, vias 0 -> 2
- net VCC: track 0.00 -> 42.8 mm, vias 0 -> 2
- net VS: track 0.00 -> 36.1 mm, vias 0 -> 2
- net HEATER_NEG: track 0.00 -> 35.0 mm, vias 0 -> 1
- net NRST: track 0.00 -> 34.0 mm, vias 0 -> 3
- net CAN_SLEEP: track 0.00 -> 33.7 mm
- net SPI1_MOSI: track 0.00 -> 31.0 mm, vias 0 -> 4
- net RCAL: track 0.00 -> 30.8 mm, vias 0 -> 1
- net HEATER_DIAG: track 0.00 -> 30.8 mm, vias 0 -> 2
- net OUT3: track 0.00 -> 28.5 mm, vias 0 -> 1
- net PUMP_I: track 0.00 -> 26.8 mm, vias 0 -> 2
- net CAN_RX: track 0.00 -> 26.6 mm, vias 0 -> 2
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Other:
- board size 56 x 25 mm -> 69.5 x 30 mm
