File: board/rev_a.sch (EAGLE design)
At the start: 52 parts, among them IC3 MCP2551, Q1 Logic level FET, X1 B4B-ZR

Commit message: Routed PCB
Parts:
- removed D3, D4: (no value), zetex:D_ACACSOT323
- removed J1, J2: (no value), SparkFun-Connectors:CONN_06LONGPADS
- removed J3: (no value), SparkFun-Connectors:CONN_04LOCK
- removed RN1, RN4: 1K, resistor-dil:4R-N0603-ARC
- removed S1: (no value), SparkFun-Switches:MOMENTARY-SWITCH-SPST-2-SMD-5.2MM
- added LED1: LED-APA102, Ai_LED:LED-APA102
- added PAD1, PAD2, PAD3, PAD4, PAD5, PAD6: WIREPADSMD5-2,5, wirepad:WIREPADSMD5-2,5
- added R22: 68K 0.1%, resistor:R-EU_R0603
- added R23: 22K 0.1%, resistor:R-EU_R0603
- added X2, X3: (no value), con-molex-micro-fit-3_0:HEADER_POS4_43045-0401
- added X5: (no value), con-molex-micro-fit-3_0:HEADER_POS2_43045-0200
- C3: device rcl:CPOL-EUE2.5-6 -> rcl:CPOL-EUE2.5-5
- IC3: value MCP2551 -> MAX3051
- OPA1: value MCP6002 -> MCP6V64; device linear:MCP602ST -> linear:MCP604ST
- Q1: value Logic level FET -> VND7NV04
- R10, R18, R19, R7: value 22K 1% -> 22K 0.1%
- R13, R16, R6: value 100K 1% -> 100K 0.1%
- R14: value 62R 1% -> 61.9R 0.1%
- R17, R20: value 66K 1% -> 68K 0.1%
Connections:
- removed net AN2: MCU.PA1-USART2RTS/ADC1/TIM2CH2
- removed net AN3: MCU.PA2-USART2TX/ADC2/TIM2CH3
- removed net BUTTON1: MCU.PC13-TAMPER-RTC, S1.1, S1.2
- removed net HEATER_POS: J2.4
- removed net N$1: Q1.G, RN3A.2, RN3B.1
- removed net N$3: RN1A.2, RN1B.1
- removed net N$9: RN1C.2, RN1D.1
- removed net OPA3_OUT: MCU.PB1-ADC9/TIM3CH4-TIM1CH3N, R6.2
- removed net OPA4_OUT: MCU.PB12-SPI2NSS/I2C2SMBAI/USART3CK/TIM1BKIN, R17.2
- removed net SCL: J3.3, MCU.PB6-I2C1SCL/TIM4CH1-USART1TX, RN1C.1
- removed net SDA: J3.4, MCU.PB7-I2C1SDA/TIM4CH2-USART1RX, RN1A.1
- new net HEATER_DIAG: MCU.PA1-USART2RTS/ADC1/TIM2CH2, Q1.G, RN3A.2, RN3B.1
- new net N$10: OPA1B.+IN, R22.2, R23.2
- new net NERST_R: MCU.PB12-SPI2NSS/I2C2SMBAI/USART3CK/TIM1BKIN, OPA1D.OUT, R17.2
- new net PUMP_I: MCU.PB1-ADC9/TIM3CH4-TIM1CH3N, OPA1C.OUT, R6.2
- new net SPI1_CS: MCU.PA15/JTDI-TIM2CH1ETR/SPI1NSS
- new net SPI1_MISO: MCU.PB4/JNTRST--TIM3CH1/SPI1MISO
- new net SPI1_MOSI: LED1.DI, MCU.PB5-I2C1SMBAI-TIM3CH2/SPI1MOSI
- new net SPI1_SCK: LED1.CI, MCU.PB3/JTDO--TIM2CH2/TRACESWO/SPI1SCK
- net 12V: now also PAD3.P, X2.2, X3.2; no longer J1.6
- net 5V: now also LED1.VCC; no longer D3.C, D4.C, IC3.VDD, J3.2
- net AN1: no longer MCU.PA0-WKUP/USART2CTS/ADC0/TIM2CH1ETR
- net DAC2: now also R15.2; no longer OPA1B.+IN
- net GND: now also LED1.GND, R23.1, X2.1, X3.1; no longer D3.A, D4.A, J1.1, J3.1, S1.3, S1.4
- net HEATER_NEG: now also PAD4.P; no longer J2.3
- net IP: now also PAD6.P; no longer J2.1
- net OPA3_IN+: now also OPA1C.+IN; no longer MCU.PB0-ADC8/TIM3CH3-TIM1CH2N
- net OPA3_IN-: now also OPA1C.-IN; no longer MCU.PB2/BOOT1
- net OPA4_IN+: no longer MCU.PB11-I2C2SDA/USART3RX-TIM2CH4
- net OPA4_IN-: no longer MCU.PB10-I2C2SCL/USART3TX-TIM2CH3
- net OUT1: now also X5.2; no longer J1.5
- net OUT2: now also X5.1; no longer J1.4
- net OUT3: now also X2.4, X3.4; no longer J1.3, RN4A.1, RN4B.1
- net OUT3_PROT: no longer D3.CA, RN4A.2, RN4B.2
- net OUT4: now also X2.3, X3.3; no longer J1.2, RN4C.1, RN4D.1
- net OUT4_PROT: no longer D4.CA, RN4C.2, RN4D.2
- net RCAL: now also PAD2.P; no longer J2.5
- net TIM1_CH1: no longer R15.2
- net VBAT: now also MCU.PA0-WKUP/USART2CTS/ADC0/TIM2CH1ETR
- net VCC: now also IC3.VDD; no longer RN1B.2, RN1D.2
- net VGND: now also MCU.PA2-USART2TX/ADC2/TIM2CH3, PAD5.P; no longer J2.2
- net VS: now also PAD1.P; no longer J2.6
Other:
- note removed: "OPA3"
- note removed: "OPA4"
- moved on the sheet: D1, D2, RN2A, RN2B, RN2C, RN2D
